Commit message: 2/7/2021

File: src/my_robot_urdf/urdf/m2wr_tw.xacro (robot description, xacro)
@@ -3,13 +3,6 @@
   <xacro:include filename="$(find my_robot_urdf)/urdf/mybot.gazebo" />
   <xacro:include filename="$(find my_robot_urdf)/urdf/materials.xacro" />
-  <!--xacro:include filename="$(find my_robot_urdf)/urdf/macros.xacro" /-->
+  <xacro:include filename="$(find my_robot_urdf)/urdf/macros.xacro" />
  <link name="link_chassis">
-    <!-- pose and inertial -->
-    <pose>0 0 0 0 0 0</pose>
-	<inertial>
-      <mass value="5"/>
-      <origin rpy="0 0 0" xyz="0 0 0"/>
-      <inertia ixx="0.0395416666667" ixy="0" ixz="0" iyy="0.106208333333" iyz="0" izz="0.106208333333"/>
-    </inertial>
     <!-- body -->
     <collision name="collision_chassis">
@@ -26,7 +19,21 @@
     </visual>
   </link>
+  <!-- Inertial link stores the robot's inertial information -->
+  <link name="inertial_link">
+    <inertial>
+      <mass value="45" />
+      <origin xyz="-0.00065 -0.085 0.062" />
+      <inertia ixx="0.6022" ixy="-0.02364" ixz="-0.1197" iyy="1.7386" iyz="-0.001544" izz="2.0296" />
+    </inertial>
+  </link>
+  <joint name="inertial_joint" type="fixed">
+    <origin xyz="0 0 0" rpy="0 0 0" />
+    <parent link="link_chassis" />
+    <child link="inertial_link" />
+  </joint>
+  <!-- Wheels and Joints -->
   <link name="link_right_wheel">
     <inertial>
-      <mass value="0.2"/>
+      <mass value="2"/>
       <origin rpy="0 1.5707 1.5707" xyz="0 0 0"/>
       <inertia ixx="0.000526666666667" ixy="0" ixz="0" iyy="0.000526666666667" iyz="0" izz="0.001"/>
@@ -43,4 +50,5 @@
         <cylinder length="0.04" radius="0.1"/>
       </geometry>
+	  <material name="black"/>
     </visual>
   </link>
@@ -55,5 +63,5 @@
   <link name="link_left_wheel">
     <inertial>
-      <mass value="0.2"/>
+      <mass value="2"/>
       <origin rpy="0 1.5707 1.5707" xyz="0 0 0"/>
       <inertia ixx="0.000526666666667" ixy="0" ixz="0" iyy="0.000526666666667" iyz="0" izz="0.001"/>
@@ -70,4 +78,5 @@
         <cylinder length="0.04" radius="0.1"/>
       </geometry>
+	  <material name="black"/>
     </visual>
   </link>
@@ -82,5 +91,5 @@
     <link name="link_back_right_wheel">
     <inertial>
-      <mass value="0.2"/>
+      <mass value="2"/>
       <origin rpy="0 1.5707 1.5707" xyz="0 0 0"/>
       <inertia ixx="0.000526666666667" ixy="0" ixz="0" iyy="0.000526666666667" iyz="0" izz="0.001"/>
@@ -97,4 +106,5 @@
         <cylinder length="0.04" radius="0.1"/>
       </geometry>
+	  <material name="black"/>
     </visual>
   </link>
@@ -109,5 +119,5 @@
     <link name="link_back_left_wheel">
     <inertial>
-      <mass value="0.2"/>
+      <mass value="2"/>
       <origin rpy="0 1.5707 1.5707" xyz="0 0 0"/>
       <inertia ixx="0.000526666666667" ixy="0" ixz="0" iyy="0.000526666666667" iyz="0" izz="0.001"/>
@@ -124,4 +134,5 @@
         <cylinder length="0.04" radius="0.1"/>
       </geometry>
+	  <material name="black"/>
     </visual>
   </link>
@@ -134,4 +145,5 @@
     <joint_properties damping="1.0" friction="1.0"/>
   </joint>
+  <!-- Camera-->
     <link name="camera">
     <collision>
@@ -160,4 +172,5 @@
     <child link="camera"/>
   </joint>
+  <!-- Lidar Scanner-->
   <link name="laser_link">
   <collision>
@@ -172,4 +185,5 @@
      <box size="0.05 0.05 0.05"/>
     </geometry>
+	<material name="white"/>
   </visual>
   <inertial>
@@ -185,4 +199,5 @@
 <child link="laser_link"/>
 </joint>
+<!-- IMU -->
   <link name="imu_link">
   <collision>
@@ -197,4 +212,5 @@
      <box size="0.025 0.025 0.025"/>
     </geometry>
+	<material name="orange"/>
   </visual>
   <inertial>
